File: KiCad/Energiezähler.kicad_pcb (KiCad board)
At the start: 2 copper layers, 42 x 49 mm, 30 parts, among them J101 Power, J102 Sensor, SW101 SW_Push, U101 DC/DC, U102 LMV393, U103 WeMos_D1_mini

Commit message: new hardware data
Parts:
- D101: value LED rot -> LED red
- D102: value LED gelb -> LED yellow
Other:
- board text added: "C"
- board text added: "E"
- board text added: "EN"
- board text added: "Vin"
- board text added: "Vout"
- board text removed: "A"
Changed lines of the file:
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@@
       (effects (font (size 1 1) (thickness 0.15)))
     )
-    (fp_text value "LED gelb" (at 0.9 -3.4) (layer "F.Fab")
+    (fp_text value "LED yellow" (at 0.1 -3.2375) (layer "F.Fab")
       (effects (font (size 1 1) (thickness 0.15)))
     )
@@
     (property "Sheetname" "")
     (attr through_hole)
-    (fp_text reference "J102" (at 2.65 4.14 90) (layer "F.SilkS")
-      (effects (font (size 1 1) (thickness 0.15)))
-    )
-    (fp_text value "Sensor" (at -2.8 3.84 90) (layer "F.Fab")
-      (effects (font (size 1 1) (thickness 0.15)))
-    )
-    (fp_text user "${REFERENCE}" (at 2.65 4.14 90) (layer "F.Fab")
+    (fp_text reference "J102" (at 3 6.8525 90) (layer "F.SilkS")
+      (effects (font (size 1 1) (thickness 0.15)))
+    )
+    (fp_text value "Sensor" (at 4.45 6.2525 90) (layer "F.Fab")
+      (effects (font (size 1 1) (thickness 0.15)))
+    )
+    (fp_text user "${REFERENCE}" (at 3 6.8525 90) (layer "F.Fab")
       (effects (font (size 1 1) (thickness 0.15)))
     )
@@
     (descr "Through hole straight pin header, 1x04, 2.54mm pitch, single row")
     (tags "Through hole pin header THT 1x04 2.54mm single row")
+    (property "Feld4" "https://www.amazon.de/PEMENOL-Einstellbar-Spannungwandler-Stromversorgung-Wirkungsgrad/dp/B07DP2MDJQ")
+    (property "Feld5" "1=Enable, 2=Vin 12V..24V, 3=GND, 4=Vout 5.0V")
     (property "Sheetfile" "Energiezähler.kicad_sch")
     (property "Sheetname" "")
     (attr through_hole)
-    (fp_text reference "U101" (at 6.55 0.3) (layer "F.SilkS")
-      (effects (font (size 1 1) (thickness 0.15)))
-    )
-    (fp_text value "DC/DC" (at 5.95 2.05) (layer "F.Fab")
-      (effects (font (size 1 1) (thickness 0.15)))
-    )
-    (fp_text user "${REFERENCE}" (at 6.55 0.3) (layer "F.Fab")
+    (fp_text reference "U101" (at 13 4.1375) (layer "F.SilkS")
+      (effects (font (size 1 1) (thickness 0.15)))
+    )
+    (fp_text value "DC/DC" (at 12.4 6.0375) (layer "F.Fab")
+      (effects (font (size 1 1) (thickness 0.15)))
+    )
+    (fp_text user "${REFERENCE}" (at 13 4.1375) (layer "F.Fab")
       (effects (font (size 1 1) (thickness 0.15)))
     )
@@
       (effects (font (size 1 1) (thickness 0.15)))
     )
-    (fp_text value "LED rot" (at 0.9 3.1) (layer "F.Fab")
+    (fp_text value "LED red" (at 0.9 3.1) (layer "F.Fab")
       (effects (font (size 1 1) (thickness 0.15)))
     )
@@
     (effects (font (size 1 1) (thickness 0.15)))
   )
+  (gr_text "Vin" (at 96.35 79.35) (layer "F.Fab")
+    (effects (font (size 1 1) (thickness 0.15)))
+  )
+  (gr_text "GND" (at 95.9 76.85) (layer "F.Fab")
+    (effects (font (size 1 1) (thickness 0.15)))
+  )
+  (gr_text "C" (at 62.5 61.7 90) (layer "F.Fab")
+    (effects (font (size 1 1) (thickness 0.15)))
+  )
+  (gr_text "Vout" (at 95.7 74.2) (layer "F.Fab")
+    (effects (font (size 1 1) (thickness 0.15)))
+  )
   (gr_text "K" (at 98 41.75) (layer "F.Fab")
     (effects (font (size 0.8 0.8) (thickness 0.2)))
   )
+  (gr_text "EN" (at 96.35 81.9) (layer "F.Fab")
+    (effects (font (size 1 1) (thickness 0.15)))
+  )
   (gr_text "K" (at 98 46.45) (layer "F.Fab")
     (effects (font (size 0.8 0.8) (thickness 0.2)))
   )
+  (gr_text "E" (at 62.5 64.2 90) (layer "F.Fab")
+    (effects (font (size 1 1) (thickness 0.15)))
+  )
+  (gr_text "GND" (at 62.45 68 90) (layer "F.Fab")
+    (effects (font (size 1 1) (thickness 0.15)))
+  )
   (gr_text "Vcc" (at 125.8 138 90) (layer "User.2")
     (effects (font (size 2 2) (thickness 0.15)))
@@
     (effects (font (size 1 1) (thickness 0.15)))
   )
-  (gr_text "K" (at 39.4 137.9 90) (layer "User.2")
+  (gr_text "C" (at 39.4 137.9 90) (layer "User.2")
     (effects (font (size 2 2) (thickness 0.15)))
   )
-  (gr_text "A" (at 39.5 129.9 90) (layer "User.2")
+  (gr_text "E" (at 39.5 129.9 90) (layer "User.2")
     (effects (font (size 2 2) (thickness 0.15)))
   )
