File: KiCad/Energiezähler.kicad_sch (KiCad schematic)
At the start: 31 parts, among them J101 Power, J102 Sensor, SW101 SW_Push, U101 DC/DC, U102 LMV393, U103 WeMos_D1_mini

Commit message: new hardware data
Parts:
- removed D0: SFH 309 FA, symbol Device:D_Photo
- added Q0: SFH309, symbol Sensor_Optical:SFH309
- D101: value LED rot -> LED red
- D102: value LED gelb -> LED yellow
- U101: Info (none) -> 1=Enable, 2=Vin 12V..24V, 3=GND, 4=Vout 5.0V
Changed lines of the file:
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@@
+    (stroke (width 0) (type default) (color 0 0 0 0))
+  )
+  (wire (pts (xy 21.59 99.06) (xy 33.02 99.06))
     (stroke (width 0) (type default) (color 0 0 0 0))
   )
@@
     (stroke (width 0) (type default) (color 0 0 0 0))
   )
+  (wire (pts (xy 21.59 111.76) (xy 33.02 111.76))
+    (stroke (width 0) (type default) (color 0 0 0 0))
+  )
   (wire (pts (xy 212.09 76.2) (xy 212.09 78.74))
     (stroke (width 0) (type default) (color 0 0 0 0))
@@
     (stroke (width 0) (type default) (color 0 0 0 0))
   )
+  (wire (pts (xy 21.59 100.33) (xy 21.59 99.06))
+    (stroke (width 0) (type default) (color 0 0 0 0))
+  )
   (wire (pts (xy 190.5 63.5) (xy 190.5 73.66))
     (stroke (width 0) (type default) (color 0 0 0 0))
@@
     (stroke (width 0) (type default) (color 0 0 0 0))
   )
+  (wire (pts (xy 21.59 110.49) (xy 21.59 111.76))
+    (stroke (width 0) (type default) (color 0 0 0 0))
+  )
   (wire (pts (xy 133.35 99.06) (xy 133.35 100.33))
     (stroke (width 0) (type default) (color 0 0 0 0))
@@
     (stroke (width 0) (type default) (color 0 0 0 0))
   )
-  (wire (pts (xy 22.86 101.6) (xy 33.02 101.6))
-    (stroke (width 0) (type default) (color 0 0 0 0))
-  )
   (wire (pts (xy 60.96 113.03) (xy 66.04 113.03))
     (stroke (width 0) (type default) (color 0 0 0 0))
@@
     (stroke (width 0) (type default) (color 0 0 0 0))
   )
-  (wire (pts (xy 33.02 109.22) (xy 33.02 106.68))
+  (wire (pts (xy 33.02 106.68) (xy 33.02 111.76))
     (stroke (width 0) (type default) (color 0 0 0 0))
   )
@@
     (stroke (width 0) (type default) (color 0 0 0 0))
   )
-  (wire (pts (xy 22.86 109.22) (xy 33.02 109.22))
-    (stroke (width 0) (type default) (color 0 0 0 0))
-  )
   (wire (pts (xy 46.99 38.1) (xy 55.88 38.1))
     (stroke (width 0) (type default) (color 0 0 0 0))
@@
     (stroke (width 0) (type default) (color 0 0 0 0))
   )
-  (wire (pts (xy 33.02 101.6) (xy 33.02 104.14))
+  (wire (pts (xy 33.02 99.06) (xy 33.02 104.14))
     (stroke (width 0) (type default) (color 0 0 0 0))
   )
@@
       (effects (font (size 1.27 1.27)) (justify right))
     )
-    (property "Value" "LED gelb" (id 1) (at 136.271 107.4424 90)
+    (property "Value" "LED yellow" (id 1) (at 136.271 107.4424 90)
       (effects (font (size 1.27 1.27)) (justify right))
     )
@@
       (effects (font (size 1.27 1.27)) (justify right))
     )
-    (property "Value" "LED rot" (id 1) (at 215.011 96.0124 90)
+    (property "Value" "LED red" (id 1) (at 215.011 96.0124 90)
       (effects (font (size 1.27 1.27)) (justify right))
     )
@@
   )
   (symbol (lib_id "Connector_Generic:Conn_01x04") (at 109.22 40.64 0) (unit 1)
-    (in_bom yes) (on_board yes) (fields_autoplaced)
+    (in_bom yes) (on_board yes)
     (property "Reference" "U101" (id 0) (at 111.252 41.0753 0)
       (effects (font (size 1.27 1.27)) (justify left))
@@
       (effects (font (size 1.27 1.27)) hide)
     )
-    (property "Datasheet" "~" (id 3) (at 109.22 40.64 0)
-      (effects (font (size 1.27 1.27)) hide)
-    )
+    (property "Datasheet" "https://www.amazon.de/PEMENOL-Einstellbar-Spannungwandler-Stromversorgung-Wirkungsgrad/dp/B07DP2MDJQ" (id 3) (at 109.22 40.64 0)
+      (effects (font (size 1.27 1.27)) hide)
+    )
+    (property "Info" "1=Enable, 2=Vin 12V..24V, 3=GND, 4=Vout 5.0V" (id 5) (at 135.89 45.72 0))
     (pin "1")
     (pin "2")
@@
     (pin "1")
   )
+  (symbol (lib_id "Sensor_Optical:SFH309") (at 19.05 105.41 0) (unit 1)
+    (in_bom yes) (on_board no) (fields_autoplaced)
+    (property "Reference" "Q0" (id 0) (at 23.9014 103.826 0)
+      (effects (font (size 1.27 1.27)) (justify left) hide)
+    )
+    (property "Value" "SFH309" (id 1) (at 23.9014 105.0945 0)
+      (effects (font (size 1.27 1.27)) (justify left))
+    )
+    (property "Footprint" "" (id 2) (at 31.242 108.966 0)
+      (effects (font (size 1.27 1.27)) hide)
+    )
+    (property "Datasheet" "http://www.osram-os.com/Graphics/XPic2/00101811_0.pdf/SFH%20309,%20SFH%20309%20FA,%20Lead%20(Pb)%20Free%20Product%20-%20RoHS%20Compliant.pdf" (id 3) (at 19.05 105.41 0)
+      (effects (font (size 1.27 1.27)) hide)
+    )
+    (pin "1")
+    (pin "2")
+  )
   (symbol (lib_id "power:GND") (at 175.26 74.93 0) (unit 1)
     (in_bom yes) (on_board yes) (fields_autoplaced)
@@
     )
     (pin "1")
-  )
-  (symbol (lib_id "Device:D_Photo") (at 22.86 106.68 90) (mirror x) (unit 1)
-    (in_bom yes) (on_board yes)
-    (property "Reference" "D0" (id 0) (at 24.8666 104.9055 90)
-      (effects (font (size 1.27 1.27)) (justify right) hide)
-    )
-    (property "Value" "SFH 309 FA" (id 1) (at 20.32 99.06 90)
-      (effects (font (size 1.27 1.27)) (justify right))
-    )
-    (property "Footprint" "" (id 2) (at 22.86 105.41 0)
-      (effects (font (size 1.27 1.27)) hide)
-    )
-    (property "Datasheet" "~" (id 3) (at 22.86 105.41 0)
-      (effects (font (size 1.27 1.27)) hide)
-    )
-    (pin "1")
-    (pin "2")
   )
   (symbol (lib_id "Device:R") (at 154.94 147.32 180) (unit 1)
@@
       (reference "C107") (unit 1) (value "47n") (footprint "Capacitor_SMD:C_0805_2012Metric_Pad1.18x1.45mm_HandSolder")
     )
-    (path "/e980477b-b392-44a9-93da-0fc4c3713127"
-      (reference "D0") (unit 1) (value "SFH 309 FA") (footprint "")
-    )
     (path "/94e2d730-4b5e-4574-94bc-3eb19f6e4dde"
-      (reference "D101") (unit 1) (value "LED rot") (footprint "LED_THT:LED_D3.0mm")
+      (reference "D101") (unit 1) (value "LED red") (footprint "LED_THT:LED_D3.0mm")
     )
     (path "/8189a27d-f1ce-459b-80e6-6e50f8ef4f05"
-      (reference "D102") (unit 1) (value "LED gelb") (footprint "LED_THT:LED_D3.0mm")
+      (reference "D102") (unit 1) (value "LED yellow") (footprint "LED_THT:LED_D3.0mm")
     )
     (path "/7b88666f-5421-4f32-8b5a-49520155d5af"
@@
       (reference "J102") (unit 1) (value "Sensor") (footprint "Connector_PinHeader_2.54mm:PinHeader_1x04_P2.54mm_Vertical")
     )
+    (path "/e0e87955-5e1d-4ea4-92a3-c84c90715914"
+      (reference "Q0") (unit 1) (value "SFH309") (footprint "")
+    )
     (path "/f4e06298-3e35-4c4f-8804-c4de85c21880"
